File: Hydrous/Hydrous.kicad_pcb (KiCad board)
At the start: 2 copper layers, 97.2 x 47.6 mm, 60 parts, among them J1 Screw_Terminal_01x02, J10 Entrada 12v, J11 Encoder, J12 PB1 (OK), J13 PB2 (RETURN), J14 Sensor de humedad, J2 Screw_Terminal_01x02, J3 Screw_Terminal_01x02, J4 Screw_Terminal_01x02, J5 Screw_Terminal_01x02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

Commit message: update
Routing:
- net VCCQ: track 245.3 -> 247.0 mm
- added copper zone on B.Cu, net GND
Changed lines of the file:
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@@
 			(at 0 4 90)
 			(layer "F.Fab")
+			(hide yes)
 			(effects
 				(font
@@
 		(model "${EASYEDA2KICAD}/easyeda2kicad.3dshapes/R0805_L2.0-W1.3-H0.6.wrl"
 			(offset
-				(xyz -1.41 -0 -0)
+				(xyz 0.09 -0 -0)
 			)
 			(scale
@@
 			)
 			(rotate
-				(xyz 0 0 0)
+				(xyz -0 -0 -0)
 			)
 		)
@@
 			(at 0 -4 90)
 			(layer "F.SilkS")
+			(hide yes)
 			(effects
 				(font
@@
 			(at 0 4 90)
 			(layer "F.Fab")
+			(hide yes)
 			(effects
 				(font
@@
 		(model "${EASYEDA2KICAD}/easyeda2kicad.3dshapes/LED0805-RD_RED.wrl"
 			(offset
-				(xyz 0 -0 -0)
+				(xyz 0 0 -0)
 			)
 			(scale
@@
 			)
 			(rotate
-				(xyz 0 0 0)
+				(xyz -0 -0 -0)
 			)
 		)
@@
 	)
 	(segment
-		(start 120.65 59.69)
-		(end 123.19 57.15)
-		(width 0.3302)
-		(layer "B.Cu")
-		(net 9)
-	)
-	(segment
 		(start 140.97 76.2)
 		(end 142.24 74.93)
@@
 	)
 	(segment
+		(start 109.22 59.69)
+		(end 123.19 59.69)
+		(width 0.3302)
+		(layer "B.Cu")
+		(net 9)
+	)
+	(segment
 		(start 138.2 38.3)
 		(end 139.2 39.3)
@@
 	)
 	(segment
-		(start 109.22 59.69)
-		(end 120.65 59.69)
+		(start 123.444 59.436)
+		(end 123.444 57.404)
 		(width 0.3302)
 		(layer "B.Cu")
@@
 	)
 	(segment
+		(start 123.19 59.69)
+		(end 123.444 59.436)
+		(width 0.3302)
+		(layer "B.Cu")
+		(net 9)
+	)
+	(segment
+		(start 123.444 57.404)
+		(end 123.19 57.15)
+		(width 0.3302)
+		(layer "B.Cu")
+		(net 9)
+	)
+	(segment
 		(start 69.5 76.445)
 		(end 73.0275 79.9725)
@@
 			)
 		)
+	)
+	(zone
+		(net 2)
+		(net_name "GND")
+		(layer "B.Cu")
+		(hatch edge 0.5)
+		(priority 1)
+		(connect_pads
+			(clearance 0.5)
+		)
+		(min_thickness 0.25)
+		(filled_areas_thickness no)
+		(fill yes
+			(thermal_gap 0.5)
+			(thermal_bridge_width 0.5)
+		)
+		(polygon
+			(pts
+				(xy 46.99 34.925) (xy 144.145 34.925) (xy 144.145 82.55) (xy 46.99 82.55)
+			)
+		)

Commit message: Update
Other:
- board text added: "ENCODER"
- board text added: "FLUJO"
- board text added: "HUMEDAD"
- board text added: "LCD"
- board text added: "Out01"
- board text added: "Out02"
- board text added: "Out03"
- board text added: "Out04"
- board text added: "Out05"
- board text added: "Out06"
- board text added: "Out07"
- board text added: "PB1(OK)"
- board text added: "PB2(BACK)"
- board text added: "Vin(12v)"
Changed lines of the file:
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@@
+		)
+	)
+	(gr_text "LCD"
+		(at 127.889 76.581 0)
+		(layer "B.SilkS")
+		(effects
+			(font
+				(size 1 1)
+				(thickness 0.1)
+			)
+			(justify left bottom mirror)
+		)
+	)
+	(gr_text "PB1(OK)"
+		(at 137.16 73.406 90)
+		(layer "B.SilkS")
+		(effects
+			(font
+				(size 1 1)
+				(thickness 0.1)
+			)
+			(justify left bottom mirror)
+		)
+	)
+	(gr_text "Out01"
+		(at 85.217 43.434 0)
+		(layer "B.SilkS")
+		(effects
+			(font
+				(size 1 1)
+				(thickness 0.1)
+			)
+			(justify left bottom mirror)
+		)
+	)
+	(gr_text "HUMEDAD"
+		(at 114.173 76.581 0)
+		(layer "B.SilkS")
+		(effects
+			(font
+				(size 1 1)
+				(thickness 0.1)
+			)
+			(justify left bottom mirror)
+		)
+	)
+	(gr_text "Out02"
+		(at 96.393 43.434 0)
+		(layer "B.SilkS")
+		(effects
+			(font
+				(size 1 1)
+				(thickness 0.1)
+			)
+			(justify left bottom mirror)
+		)
+	)
+	(gr_text "Out03"
+		(at 108.331 43.434 0)
+		(layer "B.SilkS")
+		(effects
+			(font
+				(size 1 1)
+				(thickness 0.1)
+			)
+			(justify left bottom mirror)
+		)
+	)
+	(gr_text "Out06"
+		(at 137.16 39.624 90)
+		(layer "B.SilkS")
+		(effects
+			(font
+				(size 1 1)
+				(thickness 0.1)
+			)
+			(justify left bottom mirror)
+		)
+	)
+	(gr_text "Out04"
+		(at 119.634 43.434 0)
+		(layer "B.SilkS")
+		(effects
+			(font
+				(size 1 1)
+				(thickness 0.1)
+			)
+			(justify left bottom mirror)
+		)
+	)
+	(gr_text "PB2(BACK)"
+		(at 137.16 60.96 90)
+		(layer "B.SilkS")
+		(effects
+			(font
+				(size 1 1)
+				(thickness 0.1)
+			)
+			(justify left bottom mirror)
+		)
+	)
+	(gr_text "Out05"
+		(at 131.191 43.434 0)
+		(layer "B.SilkS")
+		(effects
+			(font
+				(size 1 1)
+				(thickness 0.1)
+			)
+			(justify left bottom mirror)
+		)
+	)
+	(gr_text "Out07"
+		(at 137.16 51.816 90)
+		(layer "B.SilkS")
+		(effects
+			(font
+				(size 1 1)
+				(thickness 0.1)
+			)
+			(justify left bottom mirror)
+		)
+	)
+	(gr_text "Vin(12v)"
+		(at 74.676 43.561 0)
+		(layer "B.SilkS")
+		(effects
+			(font
+				(size 1 1)
+				(thickness 0.1)
+			)
+			(justify left bottom mirror)
+		)
+	)
+	(gr_text "ENCODER"
+		(at 96.012 76.327 0)
+		(layer "B.SilkS")
+		(effects
+			(font
+				(size 1 1)
+				(thickness 0.1)
+			)
+			(justify left bottom mirror)
+		)
+	)
+	(gr_text "FLUJO"
+		(at 76.708 74.803 0)
+		(layer "B.SilkS")
+		(effects
+			(font
+				(size 1 1)
+				(thickness 0.1)
+			)
+			(justify left bottom mirror)
 		)
 	)

Commit message: update
Other:
- board text added: "Vin(12V)"
- board text removed: "Vin(12v)"
Changed lines of the file:
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@@
 		)
 	)
-	(gr_text "Vin(12v)"
+	(gr_text "Vin(12V)"
 		(at 74.676 43.561 0)
 		(layer "B.SilkS")

Commit message: Update
Parts:
- added LED4: XL-2012SURC, easyeda2kicad:LED0805-RD_RED, F.Cu at (49.5, 41.3)
- added R7: RC0805FR-0775RL, easyeda2kicad:R0805, F.Cu at (63.8, 41.1)
- moved LED3 78.7 mm to (124.7, 58.7)
- moved R2 66.1 mm to (124.7, 53.7), turned to 90 degrees
- moved R25 15.9 mm to (74.0, 48.9), turned to 90 degrees
- moved R24 15.8 mm to (70.5, 48.9), turned to 90 degrees
- moved C3 15.0 mm to (93.8, 55.5), turned to 0 degrees
- moved D2 11.9 mm to (113.4, 71.4), turned to 180 degrees
- moved R5 10.7 mm to (70.0, 68.0), turned to -90 degrees
- moved C4 7.91 mm to (93.8, 65.9), turned to 180 degrees
- moved D4 7.32 mm to (93.7, 68.8)
- moved R23 6.85 mm to (124.6, 63.8), turned to -90 degrees
- moved C1 6.08 mm to (113.2, 68.1), turned to 180 degrees
- moved SW1 5.07 mm to (78.5, 60.3), turned to -90 degrees
- moved C6 4.69 mm to (84.5, 60.5)
- moved U2 3.29 mm to (93.8, 60.7), turned to 180 degrees
- moved C5 2.77 mm to (62.1, 70.0), turned to -90 degrees
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Connections:
- net 3V3 renamed +3.3V
- U3 pad 33: unconnected-(U3-IO40-Pad33) -> LED
Routing:
- net GND: track 134.1 -> 35.4 mm, vias 23 -> 11
- net +3.3V: track 248.7 -> 150.4 mm, vias 7 -> 4
- net Switch: track 107.7 -> 50.9 mm, vias 7 -> 3
- net VCC: track 175.6 -> 123.3 mm, vias 6 -> 4
- net Out a: track 98.1 -> 53.2 mm
- net Out 08 (SCL): track 117.9 -> 73.5 mm, vias 3 -> 2
- net Flujo: track 25.1 -> 57.4 mm, vias 4 -> 1
- net Out 07: track 107.1 -> 75.4 mm, vias 6 -> 2
- net VCCQ: track 247.0 -> 220.4 mm, vias 5 -> 0
- net Net-(U3-IO0): track 35.9 -> 10.6 mm, vias 4 -> 0
- net Out b: track 88.7 -> 64.0 mm, vias 4 -> 3
- net Out 05: track 102.4 -> 77.7 mm, vias 2 -> 6
- net OUT PB1: track 149.2 -> 125.9 mm
- net Net-(LED4-A): track 0.00 -> 14.2 mm
- net Out 09 (SDA): track 93.7 -> 79.6 mm, vias 6 -> 2
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Other:
- board size 97.2 x 47.6 mm -> 96.4 x 45.3 mm
- board text removed: "Boot"
- board text removed: "ENCODER"
- board text removed: "FLUJO"
- board text removed: "HUMEDAD"
- board text removed: "LCD"
- board text removed: "Out01"
- board text removed: "Out02"
- board text removed: "Out03"
- board text removed: "Out04"
- board text removed: "Out05"
- board text removed: "Out06"
- board text removed: "Out07"
- board text removed: "PB1(OK)"
- board text removed: "PB2(BACK)"
- board text removed: "Vin(12V)"

Commit message: update
Other:
- board text added: "Boot"
- board text added: "ENCODER"
- board text added: "FLUJO"
- board text added: "HUMEDAD"
- board text added: "LCD"
- board text added: "OUT01"
- board text added: "OUT02"
- board text added: "OUT03"
- board text added: "OUT04"
- board text added: "OUT05"
- board text added: "OUT06"
- board text added: "OUT07"
- board text added: "PB1(OK)"
- board text added: "PB2(BACK)"
- board text added: "PWR(12V)"
Changed lines of the file:
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@@
+		)
+	)
+	(gr_text "Boot"
+		(at 76.708 57.023 0)
+		(layer "F.SilkS")
+		(effects
+			(font
+				(size 1 1)
+				(thickness 0.1)
+			)
+			(justify left bottom)
+		)
+	)
+	(gr_text "OUT01"
+		(at 85.598 43.434 0)
+		(layer "B.SilkS")
+		(effects
+			(font
+				(size 1 1)
+				(thickness 0.1)
+			)
+			(justify left bottom mirror)
+		)
+	)
+	(gr_text "OUT03"
+		(at 108.585 43.434 0)
+		(layer "B.SilkS")
+		(effects
+			(font
+				(size 1 1)
+				(thickness 0.1)
+			)
+			(justify left bottom mirror)
+		)
+	)
+	(gr_text "OUT06"
+		(at 136.398 44.577 270)
+		(layer "B.SilkS")
+		(effects
+			(font
+				(size 1 1)
+				(thickness 0.1)
+			)
+			(justify left bottom mirror)
+		)
+	)
+	(gr_text "LCD"
+		(at 127.762 76.454 0)
+		(layer "B.SilkS")
+		(effects
+			(font
+				(size 1 1)
+				(thickness 0.1)
+			)
+			(justify left bottom mirror)
+		)
+	)
+	(gr_text "ENCODER"
+		(at 96.012 76.454 0)
+		(layer "B.SilkS")
+		(effects
+			(font
+				(size 1 1)
+				(thickness 0.1)
+			)
+			(justify left bottom mirror)
+		)
+	)
+	(gr_text "OUT02"
+		(at 96.901 43.434 0)
+		(layer "B.SilkS")
+		(effects
+			(font
+				(size 1 1)
+				(thickness 0.1)
+			)
+			(justify left bottom mirror)
+		)
+	)
+	(gr_text "PB1(OK)"
+		(at 136.525 79.375 270)
+		(layer "B.SilkS")
+		(effects
+			(font
+				(size 1 1)
+				(thickness 0.1)
+			)
+			(justify left bottom mirror)
+		)
+	)
+	(gr_text "FLUJO"
+		(at 76.581 74.803 0)
+		(layer "B.SilkS")
+		(effects
+			(font
+				(size 1 1)
+				(thickness 0.1)
+			)
+			(justify left bottom mirror)
+		)
+	)
+	(gr_text "OUT07"
+		(at 136.271 55.626 270)
+		(layer "B.SilkS")
+		(effects
+			(font
+				(size 1 1)
+				(thickness 0.1)
+			)
+			(justify left bottom mirror)
+		)
+	)
+	(gr_text "HUMEDAD"
+		(at 114.173 76.454 0)
+		(layer "B.SilkS")
+		(effects
+			(font
+				(size 1 1)
+				(thickness 0.1)
+			)
+			(justify left bottom mirror)
+		)
+	)
+	(gr_text "PB2(BACK)\n"
+		(at 136.398 68.961 270)
+		(layer "B.SilkS")
+		(effects
+			(font
+				(size 1 1)
+				(thickness 0.1)
+			)
+			(justify left bottom mirror)
+		)
+	)
+	(gr_text "PWR(12V)"
+		(at 75.057 43.434 0)
+		(layer "B.SilkS")
+		(effects
+			(font
+				(size 1 1)
+				(thickness 0.1)
+			)
+			(justify left bottom mirror)
+		)
+	)
+	(gr_text "OUT04"
+		(at 119.761 43.434 0)
+		(layer "B.SilkS")
+		(effects
+			(font
+				(size 1 1)
+				(thickness 0.1)
+			)
+			(justify left bottom mirror)
+		)
+	)
+	(gr_text "OUT05"
+		(at 131.445 43.434 0)
+		(layer "B.SilkS")
+		(effects
+			(font
+				(size 1 1)
+				(thickness 0.1)
+			)
+			(justify left bottom mirror)
 		)
 	)

Commit message: Update
Parts:
- moved C1 9.05 mm to (104.2, 66.8), turned to 0 degrees
- moved C2 9.01 mm to (104.1, 55.6), turned to 0 degrees
- moved D2 2.96 mm to (113.9, 68.5)
Routing:
- net Net-(D2-A): track 21.3 -> 10.0 mm, vias 2 -> 0
- net +3.3V: track 150.4 -> 158.5 mm
- net VCC: track 123.3 -> 129.5 mm
- net (no net): track 3.72 -> 0.00 mm, vias 2 -> 0
- net Out 06: track 79.2 -> 76.2 mm, vias 2 -> 4
- net GND: track 35.4 -> 38.2 mm, vias 11 -> 21
- net DN: track 7.24 -> 9.99 mm
- net Net-(U3-EN): track 46.3 -> 47.6 mm, vias 3 -> 2
- net Flujo: track 57.4 -> 58.7 mm
- net VBUS: track 31.9 -> 33.0 mm
- net Out b: track 64.0 -> 64.9 mm
- net OUT PB1: track 125.9 -> 126.8 mm
- net Humedad ADC: track 82.2 -> 82.7 mm

Commit message: update
Parts:
- added C7: CC0805KRX7R9BB104, easyeda2kicad:C0805, B.Cu at (50.8, 60.9)
- added C8: CS2012X7R105K500NRE, easyeda2kicad:C0805, B.Cu at (50.9, 58.7)

Commit message: Gerber update
Routing:
- net +3.3V: track 158.7 -> 156.9 mm, vias 4 -> 6
Changed lines of the file:
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@@
 	)
 	(segment
-		(start 107.442 68.453)
+		(start 104.025 65.036)
 		(end 105.791 66.802)
-		(width 0.381)
+		(width 0.508)
 		(layer "F.Cu")
 		(net 27)
 	)
 	(segment
-		(start 105.791 65.506)
-		(end 104.025 63.74)
-		(width 0.381)
+		(start 107.4674 68.453)
+		(end 105.8164 66.802)
+		(width 0.508)
 		(layer "F.Cu")
 		(net 27)
 	)
 	(segment
-		(start 105.791 66.802)
-		(end 105.791 65.506)
-		(width 0.381)
+		(start 107.4674 68.453)
+		(end 111.349 68.453)
+		(width 0.508)
 		(layer "F.Cu")
 		(net 27)
 	)
 	(segment
-		(start 111.349 68.453)
-		(end 107.442 68.453)
-		(width 0.381)
+		(start 105.8164 66.802)
+		(end 105.791 66.802)
+		(width 0.508)
+		(layer "F.Cu")
+		(net 27)
+	)
+	(segment
+		(start 104.025 63.74)
+		(end 104.025 65.036)
+		(width 0.508)
 		(layer "F.Cu")
 		(net 27)
@@
 	)
 	(segment
+		(start 129.5735 65.7687)
+		(end 129.54 65.7352)
+		(width 0.508)
+		(layer "F.Cu")
+		(net 44)
+	)
+	(segment
+		(start 127.9144 61.8236)
+		(end 128.6256 62.5348)
+		(width 0.508)
+		(layer "F.Cu")
+		(net 44)
+	)
+	(segment
+		(start 129.5735 67.4335)
+		(end 129.5735 65.7687)
+		(width 0.508)
+		(layer "F.Cu")
+		(net 44)
+	)
+	(segment
 		(start 88.392 59.944)
 		(end 88.392 57.15)
@@
 	)
 	(segment
+		(start 128.6256 62.5348)
+		(end 129.54 62.5348)
+		(width 0.508)
+		(layer "F.Cu")
+		(net 44)
+	)
+	(segment
 		(start 67.945 45.593)
 		(end 68.619 45.593)
@@
 	)
 	(segment
-		(start 130.10331 65.695)
-		(end 129.745 65.695)
-		(width 0.508)
-		(layer "F.Cu")
-		(net 44)
-	)
-	(segment
 		(start 133.7535 67.6765)
 		(end 139.2 62.23)
@@
 	)
 	(segment
-		(start 129.5735 65.8665)
-		(end 129.5735 67.4335)
-		(width 0.508)
-		(layer "F.Cu")
-		(net 44)
-	)
-	(segment
-		(start 130.8608 62.895)
-		(end 130.8608 64.93751)
-		(width 0.508)
-		(layer "F.Cu")
-		(net 44)
-	)
-	(segment
 		(start 92.202 55.499)
 		(end 92.695 55.992)
@@
 	)
 	(segment
-		(start 129.745 65.695)
-		(end 129.5735 65.8665)
-		(width 0.508)
-		(layer "F.Cu")
-		(net 44)
-	)
-	(segment
 		(start 70.485 47.459)
 		(end 74.041 47.459)
@@
 	)
 	(segment
-		(start 128.9858 62.895)
-		(end 130.8608 62.895)
-		(width 0.508)
-		(layer "F.Cu")
-		(net 44)
-	)
-	(segment
 		(start 92.036 68.834)
 		(end 92.036 68.746)
@@
 	)
 	(segment
-		(start 130.8608 64.93751)
-		(end 130.10331 65.695)
-		(width 0.508)
-		(layer "F.Cu")
-		(net 44)
-	)
-	(segment
-		(start 127.9144 61.8236)
-		(end 128.9858 62.895)
-		(width 0.508)
-		(layer "F.Cu")
-		(net 44)
-	)
-	(segment
 		(start 88.392 57.15)
 		(end 90.043 55.499)
@@
 	)
 	(via
+		(at 129.54 62.5348)
+		(size 0.6)
+		(drill 0.3)
+		(layers "F.Cu" "B.Cu")
+		(net 44)
+	)
+	(via
 		(at 49.784 64.008)
 		(size 0.6)
@@
 	(via
 		(at 92.202 55.499)
+		(size 0.6)
+		(drill 0.3)
+		(layers "F.Cu" "B.Cu")
+		(net 44)
+	)
+	(via
+		(at 129.54 65.7352)
 		(size 0.6)
 		(drill 0.3)
@@
 		(width 0.508)
 		(layer "B.Cu")
+		(net 44)
+	)
+	(segment
+		(start 129.54 65.7352)
+		(end 129.54 62.5348)
+		(width 0.508)
+		(layer "B.Cu")
