File: Hydrous/Hydrous.kicad_sch (KiCad schematic)
At the start: 60 parts, among them J1 Screw_Terminal_01x02, J10 Entrada 12v, J11 Encoder, J12 PB1 (OK), J13 PB2 (RETURN), J14 Sensor de humedad, J2 Screw_Terminal_01x02, J3 Screw_Terminal_01x02, J4 Screw_Terminal_01x02, J5 Screw_Terminal_01x02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

Commit message: Update
Other:
- moved on the sheet: LED3, R2
Changed lines of the file:
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@@
 	(wire
 		(pts
-			(xy 118.11 218.44) (xy 118.11 220.98)
+			(xy 91.44 264.16) (xy 91.44 266.7)
 		)
 		(stroke
@@
 	(wire
 		(pts
-			(xy 118.11 195.58) (xy 118.11 196.85)
+			(xy 91.44 241.3) (xy 91.44 242.57)
 		)
 		(stroke
@@
 	(wire
 		(pts
-			(xy 118.11 207.01) (xy 118.11 208.28)
+			(xy 91.44 252.73) (xy 91.44 254)
 		)
 		(stroke
@@
 	(global_label "3V3"
 		(shape input)
-		(at 118.11 195.58 90)
+		(at 91.44 241.3 90)
 		(fields_autoplaced yes)
 		(effects
@@
 		)
 		(property "Intersheetrefs" "${INTERSHEET_REFS}"
-			(at 118.11 189.0872 90)
+			(at 91.44 234.8072 90)
 			(effects
 				(font
@@
 	(symbol
 		(lib_id "easyeda2kicad:XL-2012SURC")
-		(at 118.11 213.36 90)
+		(at 91.44 259.08 90)
 		(unit 1)
 		(exclude_from_sim no)
@@
 		(fields_autoplaced yes)
 		(property "Reference" "LED3"
-			(at 120.65 212.8499 90)
+			(at 93.98 258.5699 90)
 			(effects
 				(font
@@
 		)
 		(property "Value" "XL-2012SURC"
-			(at 120.65 215.3899 90)
+			(at 93.98 261.1099 90)
 			(effects
 				(font
@@
 		)
 		(property "Footprint" "easyeda2kicad:LED0805-RD_RED"
-			(at 125.73 213.36 0)
+			(at 99.06 259.08 0)
 			(effects
 				(font
@@
 		)
 		(property "Datasheet" ""
-			(at 118.11 213.36 0)
+			(at 91.44 259.08 0)
 			(effects
 				(font
@@
 		)
 		(property "Description" ""
-			(at 118.11 213.36 0)
+			(at 91.44 259.08 0)
 			(effects
 				(font
@@
 		)
 		(property "LCSC Part" "C965812"
-			(at 128.27 213.36 0)
+			(at 101.6 259.08 0)
 			(effects
 				(font
@@
 	(symbol
 		(lib_id "power:GND")
-		(at 118.11 220.98 0)
+		(at 91.44 266.7 0)
 		(unit 1)
 		(exclude_from_sim no)
@@
 		(fields_autoplaced yes)
 		(property "Reference" "#PWR048"
-			(at 118.11 227.33 0)
+			(at 91.44 273.05 0)
 			(effects
 				(font
@@
 		)
 		(property "Value" "GND"
-			(at 118.11 226.06 0)
+			(at 91.44 271.78 0)
 			(effects
 				(font
@@
 		)
 		(property "Footprint" ""
-			(at 118.11 220.98 0)
+			(at 91.44 266.7 0)
 			(effects
 				(font
@@
 		)
 		(property "Datasheet" ""
-			(at 118.11 220.98 0)
+			(at 91.44 266.7 0)
 			(effects
 				(font
@@
 		)
 		(property "Description" "Power symbol creates a global label with name \"GND\" , ground"
-			(at 118.11 220.98 0)
+			(at 91.44 266.7 0)
 			(effects
 				(font
@@
 	(symbol
 		(lib_id "easyeda2kicad:RC0805FR-0775RL")
-		(at 118.11 201.93 90)
+		(at 91.44 247.65 90)
 		(unit 1)
 		(exclude_from_sim no)
@@
 		(fields_autoplaced yes)
 		(property "Reference" "R2"
-			(at 120.65 200.6599 90)
+			(at 93.98 246.3799 90)
 			(effects
 				(font
@@
 		)
 		(property "Value" "RC0805FR-0775RL"
-			(at 120.65 203.1999 90)
+			(at 93.98 248.9199 90)
 			(effects
 				(font
@@
 		)
 		(property "Footprint" "easyeda2kicad:R0805"
-			(at 125.73 201.93 0)
+			(at 99.06 247.65 0)
 			(effects
 				(font
@@
 		)
 		(property "Datasheet" "https://lcsc.com/product-detail/Chip-Resistor-Surface-Mount_75R-75R0-1_C141697.html"
-			(at 128.27 201.93 0)
+			(at 101.6 247.65 0)
 			(effects
 				(font
@@
 		)
 		(property "Description" ""
-			(at 118.11 201.93 0)
+			(at 91.44 247.65 0)
 			(effects
 				(font
@@
 		)
 		(property "LCSC Part" "C141697"
-			(at 130.81 201.93 0)
+			(at 104.14 247.65 0)
 			(effects
 				(font

Commit message: Update
Parts:
- added LED4: XL-2012SURC, easyeda2kicad:LED0805-RD_RED, symbol easyeda2kicad:XL-2012SURC
- added R7: RC0805FR-0775RL, easyeda2kicad:R0805, symbol easyeda2kicad:RC0805FR-0775RL
Connections:
- net GND: now also LED4.1 (K)
- net LED: now reaches U3.33 (IO40)
- net LED: now also R7.2
- net 3V3 renamed +3.3V
- new net: LED4.2 (A), R7.1
Other:
- moved on the sheet: C1, C2, C3, C4, D2, D4, J10, R5, U1, U2

Commit message: update
Parts:
- added C7: CC0805KRX7R9BB104, easyeda2kicad:C0805, symbol easyeda2kicad:CC0805KRX7R9BB104
- added C8: CS2012X7R105K500NRE, easyeda2kicad:C0805, symbol easyeda2kicad:CS2012X7R105K500NRE
Connections:
- net +3.3V: now also C7.2, C8.2
- net GND: now also C7.1, C8.1

Commit message: Gerber update
Other:
- moved on the sheet: D2, J1, J12, J14, J2, J3, J4, J5, J6, J7, J8, Q1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
